File: hw/carrier/carrier.kicad_pcb (KiCad board)
At the start: 2 copper layers, 80 x 71.5 mm, 70 parts, among them J1 Apple II slot, J2 iCESugar-Pro, J4 UART, U1 SN74LVC8T245, U10 74LVC1G07, U11 74LVC1G07, U12 74LVC1G07, U13 74LVC1G07, U2 74ALVC164245, U3 SN74LVC1T45, U4 74LVC541, U5 74LVC541, U6 74LVC2G17, U7 74LVC2G17, U8 74LVC1G07, U9 74LVC1G07

Commit message: hw: build_board records lib:name so update leaves unchanged parts alone
Co-Authored-By: Claude Opus 5.5 <noreply@anthropic.com>
Claude-Session: https://claude.ai/code/session_01PC4qAp59j55No7QPonkiuw
Parts:
- C1, C10, C11, C12, C13, C14, C15, C16, C17, C18, C19, C2, C20, C21, C22, C23, C24, C26, C27, C28, C3, C4, C5, C6, C7, C8, C9: footprint C_0603_1608Metric -> Capacitor_SMD:C_0603_1608Metric
- C25: footprint C_0805_2012Metric -> Capacitor_SMD:C_0805_2012Metric
- D1: footprint D_SMA -> Diode_SMD:D_SMA
- F1: footprint Fuse_1812_4532Metric -> Fuse:Fuse_1812_4532Metric
- J1: footprint AppleII_Slot_Edge -> gsnix:AppleII_Slot_Edge
- J2: footprint SODIMM200_DDR2 -> gsnix:SODIMM200_DDR2
- J4: footprint PinHeader_1x03_P2.54mm_Vertical -> Connector_PinHeader_2.54mm:PinHeader_1x03_P2.54mm_Vertical
- JP1, JP2: footprint PinHeader_1x02_P2.54mm_Vertical -> Connector_PinHeader_2.54mm:PinHeader_1x02_P2.54mm_Vertical
- R1, R10, R11, R12, R13, R14, R15, R16, R17, R18, R19, R2, R20, R21, R3, R4, R5, R6, R7, R8, R9: footprint R_0603_1608Metric -> Resistor_SMD:R_0603_1608Metric
- U1: footprint TSSOP-24_4.4x7.8mm_P0.65mm -> Package_SO:TSSOP-24_4.4x7.8mm_P0.65mm
- U10, U11, U12, U13, U8, U9, VR1: footprint SOT-23-5 -> Package_TO_SOT_SMD:SOT-23-5
- U2: footprint TSSOP-48_6.1x12.5mm_P0.5mm -> Package_SO:TSSOP-48_6.1x12.5mm_P0.5mm
- U3: footprint SOT-23-6 -> Package_TO_SOT_SMD:SOT-23-6
- U4, U5: footprint TSSOP-20_4.4x6.5mm_P0.65mm -> Package_SO:TSSOP-20_4.4x6.5mm_P0.65mm
- U6, U7: footprint SOT-363_SC-70-6 -> Package_TO_SOT_SMD:SOT-363_SC-70-6

Commit message: hw: carrier routed through Freerouting; hw-drc with netlist parity
Co-Authored-By: Claude Opus 5.5 <noreply@anthropic.com>
Claude-Session: https://claude.ai/code/session_01PC4qAp59j55No7QPonkiuw
Parts:
- moved J1 4.00 mm to (37.6, 75.5)
Routing:
- net GND: track 0.00 -> 425.5 mm, vias 0 -> 14
- net +3V3: track 0.00 -> 266.4 mm, vias 0 -> 13
- net slot_a_dir: track 0.00 -> 129.5 mm, vias 0 -> 8
- net SLOT_D5: track 0.00 -> 128.6 mm, vias 0 -> 10
- net slot_reset_n_o: track 0.00 -> 123.1 mm, vias 0 -> 3
- net +5V_MOD: track 0.00 -> 122.2 mm, vias 0 -> 3
- net +5V: track 0.00 -> 113.4 mm, vias 0 -> 7
- net SLOT_D1: track 0.00 -> 92.0 mm, vias 0 -> 4
- net SLOT_D0: track 0.00 -> 90.3 mm, vias 0 -> 6
- net slot_rdy_o: track 0.00 -> 87.7 mm, vias 0 -> 4
- net SLOT_D4: track 0.00 -> 85.0 mm, vias 0 -> 5
- net SLOT_D2: track 0.00 -> 81.7 mm, vias 0 -> 6
- net slot_dma_n_o: track 0.00 -> 78.4 mm, vias 0 -> 4
- net SLOT_D3: track 0.00 -> 67.1 mm, vias 0 -> 4
- net SLOT_IOSEL_N: track 0.00 -> 67.0 mm, vias 0 -> 2
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Other:
- board size 80 x 71.5 mm -> 80 x 75.5 mm
